Commit message: Lab 2 - Commit 2
Added center wheel; started to use joint_state_publisher_gui.

File: urdf/navvis_robot.xacro (robot description, xacro)
@@ -83,4 +83,23 @@
         <origin xyz="0.2325 0.0001 1.9201" rpy="-0.0012 0.1146 -0.0015" />
     </joint>
+    <link name="center_wheel">
+        <visual>
+            <geometry>
+                <cylinder radius="0.15" length="0.05" />
+            </geometry>
+        </visual>
+        <collision>
+            <geometry>
+                <cylinder radius="0.15" length="0.05" />
+            </geometry>
+        </collision>
+    </link>
+    <joint name="base_center_wheel_joint" type="continuous">
+        <parent link="base" />
+        <child link="center_wheel" />
+        <origin xyz="0.10 0.0 0.0" rpy="-1.5707 0.0 0.0" />
+        <axis xyz="0.0 0.025 0.0" rpy="0 0 0" />
+        <limit effort="10000" velocity="1000" />
+    </joint>
     <xacro:macro name="wheel" params="side reflect">
         <link name="${side}_wheel">
@@ -96,8 +115,10 @@
             </collision>
         </link>
-        <joint name="base_${side}_wheel" type="fixed">
+        <joint name="base_${side}_wheel" type="continuous">
             <parent link="base" />
             <child link="${side}_wheel" />
             <orgin xyz="-0.10 (${0.4 * reflect}) 0.0" rpy="-1.5707 0.0 0.0" />
+            <axis xyz="0.0 0.025 0.0" rpy="0 0 0" />
+            <limit effort="10000" velocity="1000" />
         </joint>
     </xacro:macro>

Commit message: Lab2 3rd Commit
Using gazebo_plugins and velodyne_description. Still having
troubles with robot transforms and static positioning.

File: urdf/navvis_robot.xacro (robot description, xacro)
@@ -1,4 +1,6 @@
 <?xml version="1.0"?>
 <robot name="navvis" xmlns:xacro="http://www.ros.org/wiki/xacro">
+    <xacro:include filename="$(find gazebo_plugins)/test/multi_robot_scenario/xacro/laser/hokuyo.xacro" />
+    <xacro:include filename="$(find velodyne_description)/urdf/VLP-16.urdf.xacro"/>
     <link name="base">
         <visual>
@@ -15,72 +17,10 @@
         </collision>
     </link>
-    <link name="laser_vert_bottom">
-        <visual>
-            <geometry>
-                <box size="0.062 0.062 0.087" />
-            </geometry>
-        </visual>
-        <collision>
-            <geometry>
-                <box size="0.062 0.062 0.087" />
-            </geometry>
-        </collision>
-    </link>
-    <link name="laser_vert_top_right">
-        <visual>
-            <geometry>
-                <box size="0.062 0.062 0.087" />
-            </geometry>
-        </visual>
-        <collision>
-            <geometry>
-                <box size="0.062 0.062 0.087" />
-            </geometry>
-        </collision>
-    </link>
-    <link name="laser_vert_top_left">
-        <visual>
-            <geometry>
-                <box size="0.062 0.062 0.087" />
-            </geometry>
-        </visual>
-        <collision>
-            <geometry>
-                <box size="0.062 0.062 0.087" />
-            </geometry>
-        </collision>
-    </link>
-    <link name="laser_horiz">
-        <visual>
-            <geometry>
-                <cylinder radius="0.052" length="0.072" />
-            </geometry>
-        </visual>
-        <collision>
-            <geometry>
-                <cylinder radius="0.052" length="0.072" />
-            </geometry>
-        </collision>
-    </link>
-    <joint name="base_laser_vert_bottom_joint" type="fixed">
-        <parent link="base" />
-        <child link="laser_vert_bottom" />
-        <origin xyz="0.3158 -0.0021 0.5100" rpy="3.1355 -1.3045 0.005" />
-    </joint>
-    <joint name="base_laser_vert_top_right_joint" type="fixed">
-        <parent link="base" />
-        <child link="laser_vert_top_right" />
-        <origin xyz="0.2978 -0.1450 1.8451" rpy="-1.1760 0.6313 -1.9377" />
-    </joint>
-    <joint name="base_laser_vert_top_left_joint" type="fixed">
-        <parent link="base" />
-        <child link="laser_vert_top_left" />
-        <origin xyz="0.2997 0.1531 1.8443" rpy="1.1780 0.6198 1.9560" />
-    </joint>
-    <joint name="base_laser_horiz_joint" type="fixed">
-        <parent link="base" />
-        <child link="laser_horiz" />
-        <origin xyz="0.2325 0.0001 1.9201" rpy="-0.0012 0.1146 -0.0015" />
-    </joint>
+    <xacro:laser name="laser_vert_bottom" parent="base" xyz="0.3158 -0.0021 0.5100" rpy="3.1355 -1.3045 0.005" meshes="package://gazebo_plugins/test/multi_robot_scenario/meshes/laser" />
+    <xacro:laser name="laser_vert_top_right" parent="base" xyz="0.2978 -0.1450 1.8451" rpy="-1.1760 0.6313 -1.9377" meshes="package://gazebo_plugins/test/multi_robot_scenario/meshes/laser" />
+    <xacro:laser name="laser_vert_top_left" parent="base" xyz="0.2997 0.1531 1.8443" rpy="1.1780 0.6198 1.9560" meshes="package://gazebo_plugins/test/multi_robot_scenario/meshes/laser" />
+    <xacro:VLP-16 parent="base" name="laser_horiz" topic="laser_horiz/packets" hz="10" samples="440" gpu="false">
+        <origin xyz="0.2325416305773505 -0.0001380069427607134 1.920122926231907" rpy="-0.0012068 0.114646 -0.0015308" />
+    </xacro:VLP-16>
     <link name="center_wheel">
         <visual>
@@ -99,6 +39,6 @@
         <child link="center_wheel" />
         <origin xyz="0.10 0.0 0.0" rpy="-1.5707 0.0 0.0" />
-        <axis xyz="0.0 0.025 0.0" rpy="0 0 0" />
-        <limit effort="10000" velocity="1000" />
+        <axis xyz="0.0 0.0 1.0" rpy="0 0 0" />
+        <limit effort="30" velocity="1.0" lower="-2.2" upper="0.7" />
     </joint>
     <xacro:macro name="wheel" params="side reflect">
@@ -119,6 +59,6 @@
             <child link="${side}_wheel" />
             <orgin xyz="-0.10 (${0.4 * reflect}) 0.0" rpy="-1.5707 0.0 0.0" />
-            <axis xyz="0.0 0.025 0.0" rpy="0 0 0" />
-            <limit effort="10000" velocity="1000" />
+            <axis xyz="0.0 0.0 1.0" rpy="0 0 0" />
+            <limit effort="30" velocity="1.0" lower="-2.2" upper="0.7" />
         </joint>
     </xacro:macro>
